Commit message: new things

File: fmauch_universal_robot/ur_description/urdf/inc/ur_macro.xacro (robot description, xacro)
@@ -341,13 +341,13 @@
     <link name="${prefix}tool0_inertial">
       <visual>
-    <origin xyz="0 0 0.10" />
+    <origin xyz="0 0 0.20" />
     <geometry>
-      <cylinder length="0.2" radius="0.036"/>
+      <cylinder length="0.4" radius="0.036"/>
     </geometry>
         </visual>
         <collision>
-    <origin xyz="0 0 0.10" />
+    <origin xyz="0 0 0.20" />
     <geometry>
-      <cylinder length="0.2" radius="0.036"/>
+      <cylinder length="0.4" radius="0.036"/>
     </geometry>
         </collision>
